File: DRV8874_breakout_board.kicad_pcb (KiCad board)
At the start: 2 copper layers, 20 x 25.3 mm, 17 parts, among them J1 Conn1x7, J2 Conn1x7, U1 DRV8874PWPR, U2 Logo_Small

Commit message: añadidos LCSC y archivos de produccion
Parts:
- R6: value 0 -> 10K
- R8: value 0 -> 2.49K
Changed lines of the file:
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@@
     (descr "Resistor SMD 0402 (1005 Metric), square (rectangular) end terminal, IPC_7351 nominal, (Body size source: IPC-SM-782 page 72, https://www.pcb-3d.com/wordpress/wp-content/uploads/ipc-sm-782a_amendment_1_and_2.pdf), generated with kicad-footprint-generator")
     (tags "resistor")
+    (property "LCSC" "C163478")
     (property "Sheetfile" "DRV8874_breakout_board.kicad_sch")
     (property "Sheetname" "")
@@
     (descr "Resistor SMD 0402 (1005 Metric), square (rectangular) end terminal, IPC_7351 nominal, (Body size source: IPC-SM-782 page 72, https://www.pcb-3d.com/wordpress/wp-content/uploads/ipc-sm-782a_amendment_1_and_2.pdf), generated with kicad-footprint-generator")
     (tags "resistor")
+    (property "LCSC" "C137950")
     (property "Sheetfile" "DRV8874_breakout_board.kicad_sch")
     (property "Sheetname" "")
@@
     (descr "Capacitor SMD 0603 (1608 Metric), square (rectangular) end terminal, IPC_7351 nominal, (Body size source: IPC-SM-782 page 76, https://www.pcb-3d.com/wordpress/wp-content/uploads/ipc-sm-782a_amendment_1_and_2.pdf), generated with kicad-footprint-generator")
     (tags "capacitor")
+    (property "LCSC" "C779971")
     (property "Sheetfile" "DRV8874_breakout_board.kicad_sch")
     (property "Sheetname" "")
@@
     (descr "Resistor SMD 0402 (1005 Metric), square (rectangular) end terminal, IPC_7351 nominal, (Body size source: IPC-SM-782 page 72, https://www.pcb-3d.com/wordpress/wp-content/uploads/ipc-sm-782a_amendment_1_and_2.pdf), generated with kicad-footprint-generator")
     (tags "resistor")
+    (property "LCSC" "C4044221")
     (property "Sheetfile" "DRV8874_breakout_board.kicad_sch")
     (property "Sheetname" "")
@@
     (descr "Resistor SMD 0402 (1005 Metric), square (rectangular) end terminal, IPC_7351 nominal, (Body size source: IPC-SM-782 page 72, https://www.pcb-3d.com/wordpress/wp-content/uploads/ipc-sm-782a_amendment_1_and_2.pdf), generated with kicad-footprint-generator")
     (tags "resistor")
+    (property "LCSC" "C4044221")
     (property "Sheetfile" "DRV8874_breakout_board.kicad_sch")
     (property "Sheetname" "")
@@
     (descr "Capacitor SMD 0603 (1608 Metric), square (rectangular) end terminal, IPC_7351 nominal, (Body size source: IPC-SM-782 page 76, https://www.pcb-3d.com/wordpress/wp-content/uploads/ipc-sm-782a_amendment_1_and_2.pdf), generated with kicad-footprint-generator")
     (tags "capacitor")
+    (property "LCSC" "C66501")
     (property "Sheetfile" "DRV8874_breakout_board.kicad_sch")
     (property "Sheetname" "")
@@
     (property "Sheetfile" "DRV8874_breakout_board.kicad_sch")
     (property "Sheetname" "")
-    (attr through_hole)
+    (attr through_hole exclude_from_pos_files)
     (fp_text reference "J2" (at -2.032 -0.508 -180) (layer "F.SilkS")
         (effects (font (size 0.75 0.75) (thickness 0.15)))
@@
     (property "Sheetname" "")
     (property "Size" "0402")
+    (property "dnp" "")
     (attr smd)
     (fp_text reference "R7" (at -1.52 -0.01 90) (layer "F.SilkS")
@@
     (descr "Capacitor SMD 0603 (1608 Metric), square (rectangular) end terminal, IPC_7351 nominal, (Body size source: IPC-SM-782 page 76, https://www.pcb-3d.com/wordpress/wp-content/uploads/ipc-sm-782a_amendment_1_and_2.pdf), generated with kicad-footprint-generator")
     (tags "capacitor")
+    (property "LCSC" "C66501")
     (property "Sheetfile" "DRV8874_breakout_board.kicad_sch")
     (property "Sheetname" "")
@@
     (descr "Capacitor SMD 0603 (1608 Metric), square (rectangular) end terminal, IPC_7351 nominal, (Body size source: IPC-SM-782 page 76, https://www.pcb-3d.com/wordpress/wp-content/uploads/ipc-sm-782a_amendment_1_and_2.pdf), generated with kicad-footprint-generator")
     (tags "capacitor")
+    (property "LCSC" "C66501")
     (property "Sheetfile" "DRV8874_breakout_board.kicad_sch")
     (property "Sheetname" "")
     (property "Voltage" "16v")
     (attr smd)
-    (fp_text reference "C4" (at -2.24 0) (layer "F.SilkS")
+    (fp_text reference "C4" (at -0.775 -1.29) (layer "F.SilkS")
         (effects (font (size 0.7 0.7) (thickness 0.15)))
     )
@@
     (property "Sheetfile" "DRV8874_breakout_board.kicad_sch")
     (property "Sheetname" "")
-    (attr through_hole)
+    (attr through_hole exclude_from_pos_files)
     (fp_text reference "J1" (at 2.2352 0.0508) (layer "F.SilkS")
         (effects (font (size 0.75 0.75) (thickness 0.15)))
@@
     (descr "Resistor SMD 0402 (1005 Metric), square (rectangular) end terminal, IPC_7351 nominal, (Body size source: IPC-SM-782 page 72, https://www.pcb-3d.com/wordpress/wp-content/uploads/ipc-sm-782a_amendment_1_and_2.pdf), generated with kicad-footprint-generator")
     (tags "resistor")
+    (property "LCSC" "C163478")
     (property "Sheetfile" "DRV8874_breakout_board.kicad_sch")
     (property "Sheetname" "")
@@
     (descr "Resistor SMD 0402 (1005 Metric), square (rectangular) end terminal, IPC_7351 nominal, (Body size source: IPC-SM-782 page 72, https://www.pcb-3d.com/wordpress/wp-content/uploads/ipc-sm-782a_amendment_1_and_2.pdf), generated with kicad-footprint-generator")
     (tags "resistor")
+    (property "LCSC" "C145071")
     (property "Sheetfile" "DRV8874_breakout_board.kicad_sch")
     (property "Sheetname" "")
@@
         (effects (font (size 0.75 0.75) (thickness 0.15)))
     )
-    (fp_text value "0" (at 0 1.17) (layer "F.Fab")
+    (fp_text value "2.49K" (at 0 1.17) (layer "F.Fab")
         (effects (font (size 1 1) (thickness 0.15)))
     )
@@
     (descr "Resistor SMD 0402 (1005 Metric), square (rectangular) end terminal, IPC_7351 nominal, (Body size source: IPC-SM-782 page 72, https://www.pcb-3d.com/wordpress/wp-content/uploads/ipc-sm-782a_amendment_1_and_2.pdf), generated with kicad-footprint-generator")
     (tags "resistor")
+    (property "LCSC" "C163478")
     (property "Sheetfile" "DRV8874_breakout_board.kicad_sch")
     (property "Sheetname" "")
@@
         (effects (font (size 0.75 0.75) (thickness 0.15)))
     )
-    (fp_text value "0" (at 0 1.17 90) (layer "F.Fab")
+    (fp_text value "10K" (at 0 1.17 90) (layer "F.Fab")
         (effects (font (size 1 1) (thickness 0.15)))
     )
@@
     (effects (font (size 0.75 0.75) (thickness 0.15)) (justify left bottom mirror))
   )
-  (gr_text "DVR8874 PCB01" (at 119.2784 121.0056) (layer "F.SilkS" knockout)
+  (gr_text "DVR8874 PCB01" (at 119.11 121.64) (layer "F.SilkS" knockout)
     (effects (font (size 1.2 1.2) (thickness 0.3)) (justify left bottom))
   )
